Commit message: Remove unsupported sensors

File: gym_ignition_extra_models/iCubGazeboV2_5/icub.urdf (robot description, URDF)
Before this commit: robot iCub, 189 links, 188 joints
Links:
- removed link imu_frame
Joints:
- removed joint imu_frame_fixed_joint

Commit message: Removed skin

File: gym_ignition_extra_models/iCubGazeboV2_5/icub.urdf (robot description, URDF)
Before this commit: robot iCub, 188 links, 187 joints
Links:
- removed link l_forearm_skin_0
- removed link l_forearm_skin_1
- removed link l_forearm_skin_10
- removed link l_forearm_skin_11
- removed link l_forearm_skin_12
- removed link l_forearm_skin_13
- removed link l_forearm_skin_14
- removed link l_forearm_skin_15
- removed link l_forearm_skin_16
- removed link l_forearm_skin_17
- removed link l_forearm_skin_19
- removed link l_forearm_skin_2
- removed link l_forearm_skin_22
- removed link l_forearm_skin_24
- removed link l_forearm_skin_25
- removed link l_forearm_skin_28
- removed link l_forearm_skin_29
- removed link l_forearm_skin_3
- removed link l_forearm_skin_4
- removed link l_forearm_skin_5
- removed link l_forearm_skin_6
- removed link l_forearm_skin_7
- removed link l_forearm_skin_8
- removed link l_forearm_skin_9
- removed link l_sole_skin_0
- removed link l_sole_skin_1
- removed link l_sole_skin_10
- removed link l_sole_skin_11
- removed link l_sole_skin_12
- removed link l_sole_skin_13
- removed link l_sole_skin_14
- removed link l_sole_skin_15
- removed link l_sole_skin_17
- removed link l_sole_skin_18
- removed link l_sole_skin_19
- removed link l_sole_skin_2
- removed link l_sole_skin_20
- removed link l_sole_skin_21
- removed link l_sole_skin_22
- removed link l_sole_skin_24
- removed link l_sole_skin_25
- removed link l_sole_skin_26
- removed link l_sole_skin_27
- removed link l_sole_skin_28
- removed link l_sole_skin_29
- removed link l_sole_skin_3
- removed link l_sole_skin_4
- removed link l_sole_skin_8
- removed link l_sole_skin_9
- removed link r_forearm_skin_0
- removed link r_forearm_skin_1
- removed link r_forearm_skin_10
- removed link r_forearm_skin_11
- removed link r_forearm_skin_12
- removed link r_forearm_skin_13
- removed link r_forearm_skin_14
- removed link r_forearm_skin_15
- removed link r_forearm_skin_16
- removed link r_forearm_skin_17
- removed link r_forearm_skin_19
- removed link r_forearm_skin_2
- removed link r_forearm_skin_22
- removed link r_forearm_skin_24
- removed link r_forearm_skin_25
- removed link r_forearm_skin_28
- removed link r_forearm_skin_29
- removed link r_forearm_skin_3
- removed link r_forearm_skin_4
- removed link r_forearm_skin_5
- removed link r_forearm_skin_6
- removed link r_forearm_skin_7
- removed link r_forearm_skin_8
- removed link r_forearm_skin_9
- removed link r_lower_leg_skin_0
- removed link r_lower_leg_skin_10
- removed link r_lower_leg_skin_11
- removed link r_lower_leg_skin_14
- removed link r_lower_leg_skin_15
- removed link r_lower_leg_skin_16
- removed link r_lower_leg_skin_17
- removed link r_lower_leg_skin_19
- removed link r_lower_leg_skin_20
- removed link r_lower_leg_skin_21
- removed link r_lower_leg_skin_28
- removed link r_lower_leg_skin_29
- removed link r_lower_leg_skin_3
- removed link r_lower_leg_skin_31
- removed link r_lower_leg_skin_32
- removed link r_lower_leg_skin_35
- removed link r_lower_leg_skin_36
- removed link r_lower_leg_skin_37
- removed link r_lower_leg_skin_38
- removed link r_lower_leg_skin_4
- removed link r_lower_leg_skin_41
- removed link r_lower_leg_skin_42
- removed link r_lower_leg_skin_43
- removed link r_lower_leg_skin_46
- removed link r_lower_leg_skin_47
- removed link r_lower_leg_skin_49
- removed link r_lower_leg_skin_5
- removed link r_lower_leg_skin_50
- removed link r_lower_leg_skin_51
- removed link r_lower_leg_skin_52
- removed link r_lower_leg_skin_53
- removed link r_lower_leg_skin_54
- removed link r_lower_leg_skin_55
- removed link r_lower_leg_skin_56
- removed link r_lower_leg_skin_6
- removed link r_lower_leg_skin_60
- removed link r_lower_leg_skin_61
- removed link r_lower_leg_skin_9
- removed link r_sole_skin_0
- removed link r_sole_skin_1
- removed link r_sole_skin_10
- removed link r_sole_skin_11
- removed link r_sole_skin_12
- removed link r_sole_skin_13
- removed link r_sole_skin_14
- removed link r_sole_skin_15
- removed link r_sole_skin_17
- removed link r_sole_skin_18
- removed link r_sole_skin_19
- removed link r_sole_skin_2
- removed link r_sole_skin_20
- removed link r_sole_skin_21
- removed link r_sole_skin_22
- removed link r_sole_skin_24
- removed link r_sole_skin_25
- removed link r_sole_skin_26
- removed link r_sole_skin_27
- removed link r_sole_skin_28
- removed link r_sole_skin_29
- removed link r_sole_skin_3
- removed link r_sole_skin_4
- removed link r_sole_skin_8
- removed link r_sole_skin_9
Joints:
- removed joint l_forearm_skin_0_fixed_joint
- removed joint l_forearm_skin_10_fixed_joint
- removed joint l_forearm_skin_11_fixed_joint
- removed joint l_forearm_skin_12_fixed_joint
- removed joint l_forearm_skin_13_fixed_joint
- removed joint l_forearm_skin_14_fixed_joint
- removed joint l_forearm_skin_15_fixed_joint
- removed joint l_forearm_skin_16_fixed_joint
- removed joint l_forearm_skin_17_fixed_joint
- removed joint l_forearm_skin_19_fixed_joint
- removed joint l_forearm_skin_1_fixed_joint
- removed joint l_forearm_skin_22_fixed_joint
- removed joint l_forearm_skin_24_fixed_joint
- removed joint l_forearm_skin_25_fixed_joint
- removed joint l_forearm_skin_28_fixed_joint
- removed joint l_forearm_skin_29_fixed_joint
- removed joint l_forearm_skin_2_fixed_joint
- removed joint l_forearm_skin_3_fixed_joint
- removed joint l_forearm_skin_4_fixed_joint
- removed joint l_forearm_skin_5_fixed_joint
- removed joint l_forearm_skin_6_fixed_joint
- removed joint l_forearm_skin_7_fixed_joint
- removed joint l_forearm_skin_8_fixed_joint
- removed joint l_forearm_skin_9_fixed_joint
- removed joint l_sole_skin_0_fixed_joint
- removed joint l_sole_skin_10_fixed_joint
- removed joint l_sole_skin_11_fixed_joint
- removed joint l_sole_skin_12_fixed_joint
- removed joint l_sole_skin_13_fixed_joint
- removed joint l_sole_skin_14_fixed_joint
- removed joint l_sole_skin_15_fixed_joint
- removed joint l_sole_skin_17_fixed_joint
- removed joint l_sole_skin_18_fixed_joint
- removed joint l_sole_skin_19_fixed_joint
- removed joint l_sole_skin_1_fixed_joint
- removed joint l_sole_skin_20_fixed_joint
- removed joint l_sole_skin_21_fixed_joint
- removed joint l_sole_skin_22_fixed_joint
- removed joint l_sole_skin_24_fixed_joint
- removed joint l_sole_skin_25_fixed_joint
- removed joint l_sole_skin_26_fixed_joint
- removed joint l_sole_skin_27_fixed_joint
- removed joint l_sole_skin_28_fixed_joint
- removed joint l_sole_skin_29_fixed_joint
- removed joint l_sole_skin_2_fixed_joint
- removed joint l_sole_skin_3_fixed_joint
- removed joint l_sole_skin_4_fixed_joint
- removed joint l_sole_skin_8_fixed_joint
- removed joint l_sole_skin_9_fixed_joint
- removed joint r_forearm_skin_0_fixed_joint
- removed joint r_forearm_skin_10_fixed_joint
- removed joint r_forearm_skin_11_fixed_joint
- removed joint r_forearm_skin_12_fixed_joint
- removed joint r_forearm_skin_13_fixed_joint
- removed joint r_forearm_skin_14_fixed_joint
- removed joint r_forearm_skin_15_fixed_joint
- removed joint r_forearm_skin_16_fixed_joint
- removed joint r_forearm_skin_17_fixed_joint
- removed joint r_forearm_skin_19_fixed_joint
- removed joint r_forearm_skin_1_fixed_joint
- removed joint r_forearm_skin_22_fixed_joint
- removed joint r_forearm_skin_24_fixed_joint
- removed joint r_forearm_skin_25_fixed_joint
- removed joint r_forearm_skin_28_fixed_joint
- removed joint r_forearm_skin_29_fixed_joint
- removed joint r_forearm_skin_2_fixed_joint
- removed joint r_forearm_skin_3_fixed_joint
- removed joint r_forearm_skin_4_fixed_joint
- removed joint r_forearm_skin_5_fixed_joint
- removed joint r_forearm_skin_6_fixed_joint
- removed joint r_forearm_skin_7_fixed_joint
- removed joint r_forearm_skin_8_fixed_joint
- removed joint r_forearm_skin_9_fixed_joint
- removed joint r_lower_leg_skin_0_fixed_joint
- removed joint r_lower_leg_skin_10_fixed_joint
- removed joint r_lower_leg_skin_11_fixed_joint
- removed joint r_lower_leg_skin_14_fixed_joint
- removed joint r_lower_leg_skin_15_fixed_joint
- removed joint r_lower_leg_skin_16_fixed_joint
- removed joint r_lower_leg_skin_17_fixed_joint
- removed joint r_lower_leg_skin_19_fixed_joint
- removed joint r_lower_leg_skin_20_fixed_joint
- removed joint r_lower_leg_skin_21_fixed_joint
- removed joint r_lower_leg_skin_28_fixed_joint
- removed joint r_lower_leg_skin_29_fixed_joint
- removed joint r_lower_leg_skin_31_fixed_joint
- removed joint r_lower_leg_skin_32_fixed_joint
- removed joint r_lower_leg_skin_35_fixed_joint
- removed joint r_lower_leg_skin_36_fixed_joint
- removed joint r_lower_leg_skin_37_fixed_joint
- removed joint r_lower_leg_skin_38_fixed_joint
- removed joint r_lower_leg_skin_3_fixed_joint
- removed joint r_lower_leg_skin_41_fixed_joint
- removed joint r_lower_leg_skin_42_fixed_joint
- removed joint r_lower_leg_skin_43_fixed_joint
- removed joint r_lower_leg_skin_46_fixed_joint
- removed joint r_lower_leg_skin_47_fixed_joint
- removed joint r_lower_leg_skin_49_fixed_joint
- removed joint r_lower_leg_skin_4_fixed_joint
- removed joint r_lower_leg_skin_50_fixed_joint
- removed joint r_lower_leg_skin_51_fixed_joint
- removed joint r_lower_leg_skin_52_fixed_joint
- removed joint r_lower_leg_skin_53_fixed_joint
- removed joint r_lower_leg_skin_54_fixed_joint
- removed joint r_lower_leg_skin_55_fixed_joint
- removed joint r_lower_leg_skin_56_fixed_joint
- removed joint r_lower_leg_skin_5_fixed_joint
- removed joint r_lower_leg_skin_60_fixed_joint
- removed joint r_lower_leg_skin_61_fixed_joint
- removed joint r_lower_leg_skin_6_fixed_joint
- removed joint r_lower_leg_skin_9_fixed_joint
- removed joint r_sole_skin_0_fixed_joint
- removed joint r_sole_skin_10_fixed_joint
- removed joint r_sole_skin_11_fixed_joint
- removed joint r_sole_skin_12_fixed_joint
- removed joint r_sole_skin_13_fixed_joint
- removed joint r_sole_skin_14_fixed_joint
- removed joint r_sole_skin_15_fixed_joint
- removed joint r_sole_skin_17_fixed_joint
- removed joint r_sole_skin_18_fixed_joint
- removed joint r_sole_skin_19_fixed_joint
- removed joint r_sole_skin_1_fixed_joint
- removed joint r_sole_skin_20_fixed_joint
- removed joint r_sole_skin_21_fixed_joint
- removed joint r_sole_skin_22_fixed_joint
- removed joint r_sole_skin_24_fixed_joint
- removed joint r_sole_skin_25_fixed_joint
- removed joint r_sole_skin_26_fixed_joint
- removed joint r_sole_skin_27_fixed_joint
- removed joint r_sole_skin_28_fixed_joint
- removed joint r_sole_skin_29_fixed_joint
- removed joint r_sole_skin_2_fixed_joint
- removed joint r_sole_skin_3_fixed_joint
- removed joint r_sole_skin_4_fixed_joint
- removed joint r_sole_skin_8_fixed_joint
- removed joint r_sole_skin_9_fixed_joint

Commit message: Use relative path wrt model for mesh files

File: gym_ignition_extra_models/iCubGazeboV2_5/icub.urdf (robot description, URDF)
Before this commit: robot iCub, 52 links, 51 joints
Links:
- link chest: geometry collision mesh filename=file://meshes/simmechanics/sim_sea_2-5_chest_bb_prt-binary.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 scale=0.001 0.001 0.001; visual mesh filename=file://meshes/simmechanics/sim_sea_2-5_chest_bb_prt-binary.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 scale=0.001 0.001 0.001
- link head: geometry collision mesh filename=file://meshes/simmechanics/sim_sea_2-5_head_prt-binary.stl scale=0.001 0.001 0.001; visual mesh filename=file://meshes/simmechanics/sim_sea_2-5_head_prt-binary.stl scale=0.001 0.001 0.001
- link l_ankle_1: geometry collision mesh filename=file://meshes/simmechanics/sim_sea_2-5_l_ankle_prt-binary.s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 scale=0.001 0.001 0.001; visual mesh filename=file://meshes/simmechanics/sim_sea_2-5_l_ankle_prt-binary.s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 scale=0.001 0.001 0.001
- link l_ankle_2: geometry collision mesh filename=file://meshes/simmechanics/sim_sea_2-5_l_foot_prt-binary.stl scale=0.001 0.001 0.001; visual mesh filename=file://meshes/simmechanics/sim_sea_2-5_l_foot_prt-binary.stl scale=0.001 0.001 0.001
- link l_elbow_1: geometry collision mesh filename=file://meshes/simmechanics/sim_sea_2-5_l_elbow_prosup_prt-b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 scale=0.001 0.001 0.001; visual mesh filename=file://meshes/simmechanics/sim_sea_2-5_l_elbow_prosup_prt-b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 scale=0.001 0.001 0.001
- link l_foot: geometry collision box size=0.16 0.072 0.001; visual mesh filename=file://meshes/simmechanics/sim_sea_2-5_l_sole_prt-binary.stl scale=0.001 0.001 0.001
- link l_forearm: geometry collision mesh filename=file://meshes/simmechanics/sim_sea_2-5_l_forearm_prt-binary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 scale=0.001 0.001 0.001; visual mesh filename=file://meshes/simmechanics/sim_sea_2-5_l_forearm_prt-binary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 scale=0.001 0.001 0.001
- link l_hand: geometry collision mesh filename=file://meshes/simmechanics/sim_sea_2-5_l_hand_prt-binary.stl scale=0.001 0.001 0.001; visual mesh filename=file://meshes/simmechanics/sim_sea_2-5_l_hand_prt-binary.stl scale=0.001 0.001 0.001
- link l_hip_1: geometry collision mesh filename=file://meshes/simmechanics/sim_sea_2-5_l_hip_1_prt-binary.s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 scale=0.001 0.001 0.001; visual mesh filename=file://meshes/simmechanics/sim_sea_2-5_l_hip_1_prt-binary.s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 scale=0.001 0.001 0.001
- link l_hip_2: geometry collision mesh filename=file://meshes/simmechanics/sim_sea_2-5_l_hip_2_prt-binary.s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 scale=0.001 0.001 0.001; visual mesh filename=file://meshes/simmechanics/sim_sea_2-5_l_hip_2_prt-binary.s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 scale=0.001 0.001 0.001
- link l_hip_3: geometry collision mesh filename=file://meshes/simmechanics/sim_sea_2-5_l_upper_thigh_prt-bi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 scale=0.001 0.001 0.001; visual mesh filename=file://meshes/simmechanics/sim_sea_2-5_l_upper_thigh_prt-bi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 scale=0.001 0.001 0.001
- link l_lower_leg: geometry collision mesh filename=file://meshes/simmechanics/sim_sea_2-5_l_shank_prt-binary.s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 scale=0.001 0.001 0.001; visual mesh filename=file://meshes/simmechanics/sim_sea_2-5_l_shank_prt-binary.s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 scale=0.001 0.001 0.001
- link l_shoulder_1: geometry collision mesh filename=file://meshes/simmechanics/sim_sea_2-5_l_shoulder_1_prt-bin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 scale=0.001 0.001 0.001; visual mesh filename=file://meshes/simmechanics/sim_sea_2-5_l_shoulder_1_prt-bin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 scale=0.001 0.001 0.001
- link l_shoulder_2: geometry collision mesh filename=file://meshes/simmechanics/sim_sea_2-5_l_shoulder_2_prt-bin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 scale=0.001 0.001 0.001; visual mesh filename=file://meshes/simmechanics/sim_sea_2-5_l_shoulder_2_prt-bin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 scale=0.001 0.001 0.001
- link l_shoulder_3: geometry collision mesh filename=file://meshes/simmechanics/sim_sea_2-5_l_upper_arm_prt-bina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 scale=0.001 0.001 0.001; visual mesh filename=file://meshes/simmechanics/sim_sea_2-5_l_upper_arm_prt-bina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 scale=0.001 0.001 0.001
- link l_upper_arm: geometry collision mesh filename=file://meshes/simmechanics/sim_sea_2-5_l_elbow_prt-binary.s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 scale=0.001 0.001 0.001; visual mesh filename=file://meshes/simmechanics/sim_sea_2-5_l_elbow_prt-binary.s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 scale=0.001 0.001 0.001
- link l_upper_leg: geometry collision mesh filename=file://meshes/simmechanics/sim_sea_2-5_l_thigh_prt-binary.s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 scale=0.001 0.001 0.001; visual mesh filename=file://meshes/simmechanics/sim_sea_2-5_l_thigh_prt-binary.s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 scale=0.001 0.001 0.001
- link l_wrist_1: geometry collision mesh filename=file://meshes/simmechanics/sim_sea_2-5_l_wrist_pitch_prt-bi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 scale=0.001 0.001 0.001; visual mesh filename=file://meshes/simmechanics/sim_sea_2-5_l_wrist_pitch_prt-bi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 scale=0.001 0.001 0.001
- link neck_1: geometry collision mesh filename=file://meshes/simmechanics/sim_sea_2-5_neck_1_prt-binary.stl scale=0.001 0.001 0.001; visual mesh filename=file://meshes/simmechanics/sim_sea_2-5_neck_1_prt-binary.stl scale=0.001 0.001 0.001
- link neck_2: geometry collision mesh filename=file://meshes/simmechanics/sim_sea_2-5_neck_2_prt-binary.stl scale=0.001 0.001 0.001; visual mesh filename=file://meshes/simmechanics/sim_sea_2-5_neck_2_prt-binary.stl scale=0.001 0.001 0.001
- link r_ankle_1: geometry collision mesh filename=file://meshes/simmechanics/sim_sea_2-5_r_ankle_prt-binary.s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 scale=0.001 0.001 0.001; visual mesh filename=file://meshes/simmechanics/sim_sea_2-5_r_ankle_prt-binary.s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 scale=0.001 0.001 0.001
- link r_ankle_2: geometry collision mesh filename=file://meshes/simmechanics/sim_sea_2-5_r_foot_prt-binary.stl scale=0.001 0.001 0.001; visual mesh filename=file://meshes/simmechanics/sim_sea_2-5_r_foot_prt-binary.stl scale=0.001 0.001 0.001
- link r_elbow_1: geometry collision mesh filename=file://meshes/simmechanics/sim_sea_2-5_r_elbow_prosup_prt-b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 scale=0.001 0.001 0.001; visual mesh filename=file://meshes/simmechanics/sim_sea_2-5_r_elbow_prosup_prt-b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 scale=0.001 0.001 0.001
- link r_foot: geometry collision box size=0.16 0.072 0.001; visual mesh filename=file://meshes/simmechanics/sim_sea_2-5_r_sole_prt-binary.stl scale=0.001 0.001 0.001
- link r_forearm: geometry collision mesh filename=file://meshes/simmechanics/sim_sea_2-5_r_forearm_prt-binary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 scale=0.001 0.001 0.001; visual mesh filename=file://meshes/simmechanics/sim_sea_2-5_r_forearm_prt-binary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 scale=0.001 0.001 0.001
- link r_hand: geometry collision mesh filename=file://meshes/simmechanics/sim_sea_2-5_r_hand_prt-binary.stl scale=0.001 0.001 0.001; visual mesh filename=file://meshes/simmechanics/sim_sea_2-5_r_hand_prt-binary.stl scale=0.001 0.001 0.001
- link r_hip_1: geometry collision mesh filename=file://meshes/simmechanics/sim_sea_2-5_r_hip_1_prt-binary.s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 scale=0.001 0.001 0.001; visual mesh filename=file://meshes/simmechanics/sim_sea_2-5_r_hip_1_prt-binary.s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 scale=0.001 0.001 0.001
- link r_hip_2: geometry collision mesh filename=file://meshes/simmechanics/sim_sea_2-5_r_hip_2_prt-binary.s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 scale=0.001 0.001 0.001; visual mesh filename=file://meshes/simmechanics/sim_sea_2-5_r_hip_2_prt-binary.s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 scale=0.001 0.001 0.001
- link r_hip_3: geometry collision mesh filename=file://meshes/simmechanics/sim_sea_2-5_r_upper_thigh_prt-bi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 scale=0.001 0.001 0.001; visual mesh filename=file://meshes/simmechanics/sim_sea_2-5_r_upper_thigh_prt-bi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 scale=0.001 0.001 0.001
- link r_lower_leg: geometry collision mesh filename=file://meshes/simmechanics/sim_sea_2-5_r_shank_prt-binary.s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 scale=0.001 0.001 0.001; visual mesh filename=file://meshes/simmechanics/sim_sea_2-5_r_shank_prt-binary.s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 scale=0.001 0.001 0.001
- link r_shoulder_1: geometry collision mesh filename=file://meshes/simmechanics/sim_sea_2-5_r_shoulder_1_prt-bin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 scale=0.001 0.001 0.001; visual mesh filename=file://meshes/simmechanics/sim_sea_2-5_r_shoulder_1_prt-bin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 scale=0.001 0.001 0.001
- link r_shoulder_2: geometry collision mesh filename=file://meshes/simmechanics/sim_sea_2-5_r_shoulder_2_prt-bin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 scale=0.001 0.001 0.001; visual mesh filename=file://meshes/simmechanics/sim_sea_2-5_r_shoulder_2_prt-bin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 scale=0.001 0.001 0.001
- link r_shoulder_3: geometry collision mesh filename=file://meshes/simmechanics/sim_sea_2-5_r_upper_arm_prt-bina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 scale=0.001 0.001 0.001; visual mesh filename=file://meshes/simmechanics/sim_sea_2-5_r_upper_arm_prt-bina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 scale=0.001 0.001 0.001
- link r_upper_arm: geometry collision mesh filename=file://meshes/simmechanics/sim_sea_2-5_r_elbow_prt-binary.s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 scale=0.001 0.001 0.001; visual mesh filename=file://meshes/simmechanics/sim_sea_2-5_r_elbow_prt-binary.s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 scale=0.001 0.001 0.001
- link r_upper_leg: geometry collision mesh filename=file://meshes/simmechanics/sim_sea_2-5_r_thigh_prt-binary.s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 scale=0.001 0.001 0.001; visual mesh filename=file://meshes/simmechanics/sim_sea_2-5_r_thigh_prt-binary.s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 scale=0.001 0.001 0.001
- link r_wrist_1: geometry collision mesh filename=file://meshes/simmechanics/sim_sea_2-5_r_wrist_pitch_prt-bi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 scale=0.001 0.001 0.001; visual mesh filename=file://meshes/simmechanics/sim_sea_2-5_r_wrist_pitch_prt-bi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 scale=0.001 0.001 0.001
- link root_link: geometry collision mesh filename=file://meshes/simmechanics/sim_sea_2-5_root_link_prt-binary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 scale=0.001 0.001 0.001; visual mesh filename=file://meshes/simmechanics/sim_sea_2-5_root_link_prt-binary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 scale=0.001 0.001 0.001
- link torso_1: geometry collision mesh filename=file://meshes/simmechanics/sim_sea_2-5_lap_belt_1_prt-binar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 scale=0.001 0.001 0.001; visual mesh filename=file://meshes/simmechanics/sim_sea_2-5_lap_belt_1_prt-binar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 scale=0.001 0.001 0.001
- link torso_2: geometry collision mesh filename=file://meshes/simmechanics/sim_sea_2-5_lap_belt_2_prt-binar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 scale=0.001 0.001 0.001; visual mesh filename=file://meshes/simmechanics/sim_sea_2-5_lap_belt_2_prt-binar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 scale=0.001 0.001 0.001
