Commit message: Add end effector frame to panda arm

File: gym_ignition_models/panda/panda.urdf (robot description, URDF)
Before this commit: robot panda, 13 links, 12 joints
Links:
- added link end_effector_frame, mass 0.01
Joints:
- added joint end_effector_frame_fixed_joint: type fixed, parent panda_link7, child end_effector_frame, origin xyz=0 0 0.21 rpy=0 0 -0.785398163397

Commit message: Change panda ee frame to have x pointing forward

File: gym_ignition_models/panda/panda.urdf (robot description, URDF)
Before this commit: robot panda, 14 links, 13 joints
Joints:
- joint end_effector_frame_fixed_joint: origin xyz=0 0 0.21 rpy=0 0 -0.785398163397 -> xyz=0 0 0.21 rpy=3.14159 -1.57079 -0.785398163397
