Commit message: Improve primitive shapes of iCub model with simple collisions

File: gym_ignition_models/iCubGazeboSimpleCollisionsV2_5/icub_simple_collisions.urdf (robot description, URDF)
Before this commit: robot iCubGazeboSimpleCollisionsV2_5, 52 links, 51 joints
Links:
- link chest: geometry collision box size=0.15 0.18 0.26; visual mesh filename=file://meshes/simmechanics/sim_sea_2-5_chest_bb_prt-binary.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 scale=0.001 0.001 0.001
- link head: geometry collision sphere radius=0.11; visual mesh filename=file://meshes/simmechanics/sim_sea_2-5_head_prt-binary.stl scale=0.001 0.001 0.001
- link l_forearm: geometry collision cylinder length=0.12 radius=0.04; visual mesh filename=file://meshes/simmechanics/sim_sea_2-5_l_forearm_prt-binary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 scale=0.001 0.001 0.001
- link l_hand: geometry collision box size=0.14 0.05 0.07; visual mesh filename=file://meshes/simmechanics/sim_sea_2-5_l_hand_prt-binary.stl scale=0.001 0.001 0.001
- link l_lower_leg: geometry collision cylinder length=0.20 radius=0.056; visual mesh filename=file://meshes/simmechanics/sim_sea_2-5_l_shank_prt-binary.s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 scale=0.001 0.001 0.001
- link l_upper_arm: geometry collision cylinder length=0.13 radius=0.047; visual mesh filename=file://meshes/simmechanics/sim_sea_2-5_l_elbow_prt-binary.s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 scale=0.001 0.001 0.001
- link l_upper_leg: geometry collision cylinder length=0.16 radius=0.06; visual mesh filename=file://meshes/simmechanics/sim_sea_2-5_l_thigh_prt-binary.s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 scale=0.001 0.001 0.001
- link r_forearm: geometry collision cylinder length=0.12 radius=0.04; visual mesh filename=file://meshes/simmechanics/sim_sea_2-5_r_forearm_prt-binary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 scale=0.001 0.001 0.001
- link r_hand: geometry collision box size=0.14 0.05 0.07; visual mesh filename=file://meshes/simmechanics/sim_sea_2-5_r_hand_prt-binary.stl scale=0.001 0.001 0.001
- link r_lower_leg: geometry collision cylinder length=0.20 radius=0.056; visual mesh filename=file://meshes/simmechanics/sim_sea_2-5_r_shank_prt-binary.s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 scale=0.001 0.001 0.001
- link r_upper_arm: geometry collision cylinder length=0.13 radius=0.047; visual mesh filename=file://meshes/simmechanics/sim_sea_2-5_r_elbow_prt-binary.s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 scale=0.001 0.001 0.001
- link r_upper_leg: geometry collision cylinder length=0.16 radius=0.06; visual mesh filename=file://meshes/simmechanics/sim_sea_2-5_r_thigh_prt-binary.s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 scale=0.001 0.001 0.001
- link root_link: geometry collision box size=0.13 0.2 0.13; visual mesh filename=file://meshes/simmechanics/sim_sea_2-5_root_link_prt-binary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 scale=0.001 0.001 0.001
